File: m922.sch (KiCad schematic (older format))
At the start: 12 parts, among them J1 Conn_01x02, J2 Conn_01x02, J3 Conn_01x02, J4 Conn_01x02, J5 Conn_01x02, J6 Conn_01x02

Commit message: 試作第一案
Parts:
- removed C2, C3: 10μF/25V, Capacitor_SMD:C_1206_3216Metric_Pad1.42x1.75mm_HandSolder, symbol Device:C_Small
- removed D2, D3: MB10F-13, DIOB_MB10F-13, symbol mb10f:MB10F-13
- removed J1, J2, J3, J4, J5, J6: Conn_01x02, Connector_JST:JST_XH_B2B-XH-AM_1x02_P2.50mm_Vertical, symbol Connector_Generic:Conn_01x02
- added J1: PIEZZO, HOLLY:LDT0-028K_MID, symbol Connector:Conn_01x02_Male
- added J2: A/D CONV, Connector_JST:JST_XH_S2B-XH-A-1_1x02_P2.50mm_Horizontal, symbol Connector:Conn_01x02_Male
- D1: value MB10F-13 -> MB10F; symbol mb10f:MB10F-13 -> Diode_Bridge:B125R
Connections:
- net at D1.2 (~~): now also J1.1 (Pin_1)
- net at D1.4 (~~): now also J1.2 (Pin_2)
- net at D1.1 (+): now also C1.2, J2.2 (Pin_2); no longer C1.1
- net GND: no longer names the net of D1.3 (-)
- net GND: now also C1.1, J2.1 (Pin_1); no longer C1.2
Other:
- moved on the sheet: C1

Commit message: Rev.1 PCBGOGO ordering data
Parts:
- added TP1, TP2, TP3, TP4: TestPoint, symbol Connector:TestPoint
Connections:
- net at C1.2, D1.1 (+), J2.2 (Pin_2): now also TP2.1, TP4.1
- net at C1.1, D1.3 (-), J2.1 (Pin_1): now also TP1.1, TP3.1
Changed lines of the file:
@@
 	5350 3550 4650 3550
 Wire Wire Line
-	5350 3550 6600 3550
+	5350 3550 5950 3550
 Connection ~ 5350 3550
 Wire Wire Line
@@
 	6500 3650 6500 3900
 Wire Wire Line
-	6500 3900 5350 3900
+	6500 3900 6250 3900
 Connection ~ 5350 3900
 $Comp
@@
 	1    0    0    -1
 $EndComp
+$Comp
+L Connector:TestPoint TP3
+U 1 1 6146B9BF
+P 6050 3350
+F 0 "TP3" H 6108 3468 50  0000 L CNN
+F 1 "TestPoint" H 6108 3377 50  0000 L CNN
+F 2 "" H 6250 3350 50  0001 C CNN
+F 3 "~" H 6250 3350 50  0001 C CNN
+	1    6050 3350
+	1    0    0    -1
+$EndComp
+$Comp
+L Connector:TestPoint TP1
+U 1 1 6146BFC3
+P 5950 3100
+F 0 "TP1" H 6008 3218 50  0000 L CNN
+F 1 "TestPoint" H 6008 3127 50  0000 L CNN
+F 2 "" H 6150 3100 50  0001 C CNN
+F 3 "~" H 6150 3100 50  0001 C CNN
+	1    5950 3100
+	1    0    0    -1
+$EndComp
+$Comp
+L Connector:TestPoint TP2
+U 1 1 6146DDCC
+P 6150 4300
+F 0 "TP2" H 6092 4326 50  0000 R CNN
+F 1 "TestPoint" H 6092 4417 50  0000 R CNN
+F 2 "" H 6350 4300 50  0001 C CNN
+F 3 "~" H 6350 4300 50  0001 C CNN
+	1    6150 4300
+	-1   0    0    1
+$EndComp
+$Comp
+L Connector:TestPoint TP4
+U 1 1 6146DDD2
+P 6250 4050
+F 0 "TP4" H 6192 4076 50  0000 R CNN
+F 1 "TestPoint" H 6192 4167 50  0000 R CNN
+F 2 "" H 6450 4050 50  0001 C CNN
+F 3 "~" H 6450 4050 50  0001 C CNN
+	1    6250 4050
+	-1   0    0    1
+$EndComp
+Wire Wire Line
+	5950 3100 5950 3550
+Connection ~ 5950 3550
+Wire Wire Line
+	5950 3550 6050 3550
+Wire Wire Line
+	6050 3350 6050 3550
+Connection ~ 6050 3550
+Wire Wire Line
+	6050 3550 6600 3550
+Wire Wire Line
+	6150 4300 6150 3900
+Connection ~ 6150 3900
+Wire Wire Line
+	6150 3900 5350 3900
+Wire Wire Line
+	6250 4050 6250 3900
+Connection ~ 6250 3900
+Wire Wire Line
+	6250 3900 6150 3900
 $EndSCHEMATC
